File: hardware/SCH_PCB/My_Smart_Home_Rev2.sch (EAGLE design)
At the start: 68 parts, among them J1 ISP0, J2 ISP1, J3 MICROUSB-5P, J4 JUMPER, J5 13F-60FGYDPNW2NL, Q1 CJ2302, SW2 SW-2, U1 ATMEGA8U2, U2 ATMEGAXX8-AU, U3 W5100, U4 AMS1117, U5 W25QXX150MIL, U6 W25QXX208MIL, X1 16MHz, X2 12MHz, X3 25MHz

Commit message: Update sch and add PCB file, HW Version: Alpha2
Parts:
- added ANT1: 2.4G_ANT1, Hell-Prototypes:2.4G_ANT1
- added C10, C21: 22pF, Hell-Prototypes:C-NP
- added C25, C31: 33nF, Hell-Prototypes:C-NP
- added C27, C28, C5, C9: 0.1uF, Hell-Prototypes:C-NP
- added C30: 2.2nF, Hell-Prototypes:C-NP
- added L3, L4, L5: 8.2nH, Hell-Prototypes:L
- added R23: 22K, Hell-Prototypes:RES
- added R8, R9: 2K, Hell-Prototypes:RES
- added U7: LM75, Hell-Prototypes:LM75
- added U8: BMP180, Hell-Prototypes:BMP180
- added U9: NRF24L01P, Hell-Prototypes:NRF24L01P
- added X4: 16MHz, Hell-Prototypes:CRYSTAL
Connections:
- removed net N$21: J3.SH1, J3.SH2, J3.SH3, J3.SH4, J3.SH5, J3.SH6
- new net N$12: C21.2, U9.XC1, X4.1
- new net N$13: L3.1, L4.1, U9.ANT2
- new net N$25: R23.2, U9.IREF
- new net N$27: C25.1, U9.DVDD
- new net N$29: L3.2, L5.2, U9.ANT1
- new net N$30: C30.2, L5.1, U9.VDD_PA
- new net N$32: ANT1.1, C31.1
- new net N$34: C31.2, L4.2
- new net N$6: C10.2, U9.XC2, X4.2
- net +3V3: now also C27.2, C28.2, C5.2, C9.2, R8.2, R9.2, U7.VCC, U8.VDD, U8.VDDIO, U9.VDD1, U9.VDD2, U9.VDD3
- net AD2: now also U9.CSN
- net AD3: now also U9.CE; no longer J4.2
- net AD4/SDA: now also R9.1, U7.SDA, U8.SDA
- net AD5/SCL: now also R8.1, U7.SCL, U8.SCL
- net GND: now also ANT1.2, C10.1, C21.1, C25.2, C27.1, C28.1, C30.1, C5.1, C9.1, J3.SH1, J3.SH2, J3.SH3, J3.SH4, J3.SH5, J3.SH6, R23.1, U7.A0, U7.A1, U7.A2, U7.GND, U8.GND, U9.VSS1, U9.VSS2, U9.VSS3, U9.VSS4
- net IO8: now also R11.1
- net IO9: now also J4.2; no longer R11.1
- net MISO_1: now also U9.MISO
- net MOSI_1: now also U9.MOSI
- net SCK_1: now also U9.SCK
Other:
- note added: "My Smart Home Project Platform V2.0"
- note added: "Optional"
- note removed: "My Smart Home Project Hardware"
